File: ATAPIMega.sch (KiCad schematic (older format))
At the start: 26 parts, among them J2 IDE, U1 ATmega2560-16AU

Commit message: Add PCB
Parts:
- removed C2: 22uF, Capacitor_SMD:C_0805_2012Metric, symbol Device:C
- removed C? (x2): 20p, Capacitor_SMD:C_0402_1005Metric, symbol Device:C
- added C1, C14, C3: 22pF, Capacitor_SMD:C_0402_1005Metric, symbol Device:C
- added C10, C12, C13, C9: 22uF, Capacitor_SMD:C_0805_2012Metric, symbol Device:C
- added C11: 100nF, Capacitor_SMD:C_0402_1005Metric, symbol Device:C
- added C15: 2200uF 16V, Capacitor_THT:CP_Radial_D13.0mm_P5.00mm, symbol Device:CP
- added J5: Drive_Power, TerminalBlock_RND:TerminalBlock_RND_205-00003_1x04_P5.00mm_Horizontal, symbol Connector:Screw_Terminal_01x04
- added J6: 12V DC-In, ATAPIMega:BarrelJack_DC-005-2.0_C16214, symbol Connector:Barrel_Jack_Switch
- added J7: External buttons, Connector_PinHeader_2.54mm:PinHeader_1x08_P2.54mm_Vertical, symbol Connector_Generic:Conn_01x08
- added J?: 3.5mm, Connector_Audio:Jack_3.5mm_CUI_SJ1-3535NG_Horizontal, symbol Connector:AudioJack3
- added J?: Audio in, Connector_PinHeader_2.54mm:PinHeader_1x04_P2.54mm_Vertical, symbol Connector_Generic:Conn_01x04
- added L1: 4.7uH, Inductor_SMD:L_Bourns_SRP7028A_7.3x6.6mm, symbol Device:L
- added R10: 30k, Resistor_SMD:R_0603_1608Metric, symbol Device:R
- added R4, R5: 4.7k, Resistor_SMD:R_0402_1005Metric, symbol Device:R
- added R8: 75R, Resistor_SMD:R_0402_1005Metric, symbol Device:R
- added R9: 220k, Resistor_SMD:R_0603_1608Metric, symbol Device:R
- added RN1, RN2, RN3, RN4, RN5, RN6: 33R, Resistor_SMD:R_Array_Convex_4x0402, symbol Device:R_Pack04
- added SW1: Rew, Button_Switch_SMD:SW_Push_1P1T_NO_6x6mm_H9.5mm, symbol Switch:SW_Push
- added SW2: Prev, Button_Switch_SMD:SW_Push_1P1T_NO_6x6mm_H9.5mm, symbol Switch:SW_Push
- added SW3: Play/Pause, Button_Switch_SMD:SW_Push_1P1T_NO_6x6mm_H9.5mm, symbol Switch:SW_Push
- added SW4: Fwd, Button_Switch_SMD:SW_Push_1P1T_NO_6x6mm_H9.5mm, symbol Switch:SW_Push
- added SW5: Next, Button_Switch_SMD:SW_Push_1P1T_NO_6x6mm_H9.5mm, symbol Switch:SW_Push
- added SW6: Stop/Eject, Button_Switch_SMD:SW_Push_1P1T_NO_6x6mm_H9.5mm, symbol Switch:SW_Push
- added SW7: Shuffle/Repeat, Button_Switch_SMD:SW_Push_1P1T_NO_6x6mm_H9.5mm, symbol Switch:SW_Push
- added U3: SY8113B, Package_TO_SOT_SMD:TSOT-23-6, symbol Silergy:SY8113B
- J1: renamed from J?; footprint (none) -> Connector_IDC:IDC-Header_2x03_P2.54mm_Vertical; LCSC (none) -> C11214
- J3: renamed from J?; footprint (none) -> Connector_PinHeader_2.54mm:PinHeader_1x06_P2.54mm_Vertical; LCSC (none) -> C37208
- J4: renamed from J?; value Conn_01x04 -> OLED SSD1306; footprint (none) -> Connector_PinHeader_2.54mm:PinHeader_1x04_P2.54mm_Vertical
- gave numbers to parts that had none: 12
Connections:
- net OLED_GND is gone; now on net GND: J4.1 (Pin_1)
- net +5V: now also C12.1, C13.1, C14.1, J5.1 (Pin_1), L1.2, R4.1, R5.2, R9.1
- net CS0: now also RN2.1 (R1.1); no longer J2.37 (Pin_37)
- net D0: now also RN1.4 (R4.1); no longer J2.17 (Pin_17)
- net D1: now also RN1.3 (R3.1); no longer J2.15 (Pin_15)
- net D10: now also RN5.3 (R3.1); no longer J2.8 (Pin_8)
- net D11: now also RN5.4 (R4.1); no longer J2.10 (Pin_10)
- net D12: now also RN6.5 (R4.2); no longer J2.12 (Pin_12)
- net D13: now also RN6.6 (R3.2); no longer J2.14 (Pin_14)
- net D14: now also RN6.7 (R2.2); no longer J2.16 (Pin_16)
- net D15: now also RN6.8 (R1.2); no longer J2.18 (Pin_18)
- net D2: now also RN1.2 (R2.1); no longer J2.13 (Pin_13)
- net D3: now also RN1.1 (R1.1); no longer J2.11 (Pin_11)
- net D4: now also RN3.4 (R4.1); no longer J2.9 (Pin_9)
- net D5: now also RN3.3 (R3.1); no longer J2.7 (Pin_7)
- net D6: now also RN3.2 (R2.1); no longer J2.5 (Pin_5)
- net D7: now also RN3.1 (R1.1); no longer J2.3 (Pin_3), R6.2
- net D8: now also RN5.1 (R1.1); no longer J2.4 (Pin_4)
- net D9: now also RN5.2 (R2.1); no longer J2.6 (Pin_6)
- net DA0: now also U1.6 (PE4), RN2.2 (R2.1); no longer J2.35 (Pin_35), U1.45 (PD2)
- net DA1: now also U1.5 (PE3), RN2.3 (R3.1); no longer J2.33 (Pin_33), U1.44 (PD1)
- net DA2: now also U1.4 (PE2); no longer U1.43 (PD0)
- net DMA_RQ: now also RN4.4 (R4.1); no longer J2.21 (Pin_21), R18.1
- net FTDI_DTR: now also R8.1
- net GND: now also C1.1, C10.2, C12.2, C13.2, C15.2, C3.2, C9.2, J5.2 (Pin_2), J5.3 (Pin_3), J6.2, J7.8 (Pin_8), R10.2, SW1.1, SW2.1, SW3.1, SW4.1, SW5.1, SW6.1, SW7.1, U3.2 (GND)
- net IOR: now also RN4.2 (R2.1); no longer J2.25 (Pin_25)
- net IOW: now also RN4.3 (R3.1); no longer J2.23 (Pin_23)
- net IO_CH_RD: now also RN4.1 (R1.1); no longer J2.27 (Pin_27), R7.2
- net IRQ: now also RN2.4 (R4.1); no longer J2.31 (Pin_31), R16.1
- net ISP_RST: now also R8.2
- net OLED_SCL: now also U1.43 (PD0), R5.1
- net OLED_SDA: now also U1.44 (PD1), R4.2
- net RESET: now also U1.59 (PC6)
- net at U1.33 (XTAL2): now also Y1.1, C3.1; no longer Y1.3
- net at U1.34 (XTAL1): now also Y1.3, C1.2; no longer Y1.1
- net BTN_PREV: now reaches U1.71 (PA7)
- net BTN_PREV: now also J7.1 (Pin_1), SW2.2
- net BTN_REW: now reaches U1.72 (PA6)
- net BTN_REW: now also J7.2 (Pin_2), SW1.2
- net BTN_PLAY: now reaches U1.73 (PA5)
- net BTN_PLAY: now also J7.3 (Pin_3), SW3.2
- net BTN_FWD: now reaches U1.74 (PA4)
- net BTN_FWD: now also J7.4 (Pin_4), SW4.2
- net BTN_NEXT: now reaches U1.75 (PA3)
- net BTN_NEXT: now also J7.5 (Pin_5), SW5.2
- net BTN_SHUFFLE: now reaches U1.76 (PA2)
- net BTN_SHUFFLE: now also J7.7 (Pin_7), SW7.2
- net BTN_STOP: now reaches U1.78 (PA0)
- net BTN_STOP: now also J7.6 (Pin_6), SW6.2
- net OLED_VCC renamed OLED_5V
- new net: J2.10 (Pin_10), RN5.5 (R4.2)
- new net: J2.11 (Pin_11), RN1.8 (R1.2)
- new net: J2.12 (Pin_12), RN6.4 (R4.1)
- new net: J2.13 (Pin_13), RN1.7 (R2.2)
- new net: J2.14 (Pin_14), RN6.3 (R3.1)
- new net: J2.15 (Pin_15), RN1.6 (R3.2)
- new net: J2.16 (Pin_16), RN6.2 (R2.1)
- new net: J2.17 (Pin_17), RN1.5 (R4.2)
- new net: J2.18 (Pin_18), RN6.1 (R1.1)
- new net: J2.23 (Pin_23), RN4.6 (R3.2)
- new net: J2.25 (Pin_25), RN4.7 (R2.2)
- new net: J2.33 (Pin_33), RN2.6 (R3.2)
- new net: J2.35 (Pin_35), RN2.7 (R2.2)
- new net: J2.37 (Pin_37), RN2.8 (R1.2)
- new net: J2.4 (Pin_4), RN5.8 (R1.2)
- new net: J2.5 (Pin_5), RN3.7 (R2.2)
- new net: J2.6 (Pin_6), RN5.7 (R2.2)
- new net: J2.7 (Pin_7), RN3.6 (R3.2)
- new net: J2.8 (Pin_8), RN5.6 (R3.2)
- new net: J2.9 (Pin_9), RN3.5 (R4.2)
- new net: C11.2, U3.1 (BS)
- new net: C14.2, R10.1, R9.2, U3.3 (FB)
- new net: C11.1, L1.1, U3.6 (LX)
- new net: J?.1 (Pin_1), J?.R
- new net: J?.2 (Pin_2), J?.3 (Pin_3), J?.S
- new net: J?.4 (Pin_4), J?.T
- new net +12V: C10.1, C15.1, C9.1, J5.4 (Pin_4), J6.1, U3.4 (EN), U3.5 (IN)
- new net ATA_D7: J2.3 (Pin_3), R6.2, RN3.8 (R1.2)
- new net ATA_DMA_RQ: J2.21 (Pin_21), R18.1, RN4.5 (R4.2)
- new net ATA_IO_CH_RD: J2.27 (Pin_27), R7.2, RN4.8 (R1.2)
- new net ATA_IRQ: J2.31 (Pin_31), R16.1, RN2.5 (R4.2)
- no-connect marks 4 -> 6
Other:
- note added: "Attribution\nBackside Image"
- note removed: "Decoupling\nButtons\nSSD1306\nStep-Down\n\nPower Output\n"
- note removed: "Prev - Rew - Play/Pause - Fwd - Next - Stop - Eject - Shuffle/Repeat"
- moved on the sheet: C4, H1, H2, R2, RV1, U2

Commit message: PCB
Parts:
- added C2: 100nF, Capacitor_SMD:C_0402_1005Metric, symbol Device:C
- added H3: Catboy, ATAPIMega:catboy, symbol Mechanical:MountingHole
- J5: LCSC (none) -> C192779
- gave numbers to parts that had none: 2
Connections:
- net +5V: now also C2.2
- net GND: now also J6.3, C2.1
- no-connect marks 6 -> 5
Changed lines of the file:
@@
 F 2 "TerminalBlock_RND:TerminalBlock_RND_205-00003_1x04_P5.00mm_Horizontal" H 8650 3650 50  0001 C CNN
 F 3 "~" H 8650 3650 50  0001 C CNN
+F 4 "C192779" V 8650 3650 50  0001 C CNN "LCSC"
 	1    8650 3650
 	0    -1   -1   0
@@
 	5500 6950 5750 6950
 Connection ~ 5500 6950
-NoConn ~ 5050 7100
 $Comp
 L Device:R_Pack04 RN6
@@
 	6600 4450 6050 4450
 $Comp
-L Connector:AudioJack3 J?
+L Connector:AudioJack3 J8
 U 1 1 6254C307
 P 9250 900
-F 0 "J?" H 9232 1225 50  0000 C CNN
+F 0 "J8" H 9232 1225 50  0000 C CNN
 F 1 "3.5mm" H 9232 1134 50  0000 C CNN
 F 2 "Connector_Audio:Jack_3.5mm_CUI_SJ1-3535NG_Horizontal" H 9250 900 50  0001 C CNN
@@
 $EndComp
 $Comp
-L Connector_Generic:Conn_01x04 J?
+L Connector_Generic:Conn_01x04 J9
 U 1 1 625673FD
 P 10050 900
-F 0 "J?" H 10130 892 50  0000 L CNN
+F 0 "J9" H 10130 892 50  0000 L CNN
 F 1 "Audio in" H 10130 801 50  0000 L CNN
 F 2 "Connector_PinHeader_2.54mm:PinHeader_1x04_P2.54mm_Vertical" H 10050 900 50  0001 C CNN
@@
 Wire Wire Line
 	9700 800  9850 800
+Wire Wire Line
+	5050 7100 5200 7100
+Wire Wire Line
+	5200 7100 5200 7200
+Connection ~ 5200 7200
+$Comp
+L Device:C C2
+U 1 1 626B269E
+P 5350 1000
+F 0 "C2" V 5098 1000 50  0000 C CNN
+F 1 "100nF" V 5189 1000 50  0000 C CNN
+F 2 "Capacitor_SMD:C_0402_1005Metric" H 5388 850 50  0001 C CNN
+F 3 "https://datasheet.lcsc.com/szlcsc/Samsung-Electro-Mechanics-CL05B104KO5NNNC_C1525.pdf" H 5350 1000 50  0001 C CNN
+F 4 " C1525" V 5350 1000 50  0001 C CNN "LCSC"
+	1    5350 1000
+	-1   0    0    1
+$EndComp
+Wire Wire Line
+	5350 850  5100 850
+Connection ~ 5100 850
+Wire Wire Line
+	5100 1150 5350 1150
+Connection ~ 5100 1150
+$Comp
+L Mechanical:MountingHole H3
+U 1 1 62729D3C
+P 10650 1000
+F 0 "H3" H 10750 1046 50  0000 L CNN
+F 1 "Catboy" H 10750 955 50  0000 L CNN
+F 2 "ATAPIMega:catboy" H 10650 1000 50  0001 C CNN
+F 3 "~" H 10650 1000 50  0001 C CNN
+	1    10650 1000
+	1    0    0    -1
+$EndComp
 $EndSCHEMATC
