File: ATAPIMega.kicad_pcb (KiCad board)
At the start: 2 copper layers, 3 parts, among them J2 IDE

Commit message: Add PCB
Parts:
- added C1: 22pF, Capacitor_SMD:C_0402_1005Metric, F.Cu at (93.7, 42.2)
- added C10: 22uF, Capacitor_SMD:C_0805_2012Metric, F.Cu at (55.5, 50.8)
- added C11: 100nF, Capacitor_SMD:C_0402_1005Metric, F.Cu at (59.7, 48.0)
- added C12: 22uF, Capacitor_SMD:C_0805_2012Metric, F.Cu at (58.5, 46.2)
- added C13: 22uF, Capacitor_SMD:C_0805_2012Metric, F.Cu at (58.5, 44.2)
- added C14: 22pF, Capacitor_SMD:C_0402_1005Metric, F.Cu at (55.9, 54.9)
- added C15: 2200uF 16V, Capacitor_THT:CP_Radial_D13.0mm_P5.00mm, F.Cu at (48.5, 44.7)
- added C3: 22pF, Capacitor_SMD:C_0402_1005Metric, F.Cu at (99.2, 42.2)
- added C4: 100nF, Capacitor_SMD:C_0402_1005Metric, F.Cu at (100.2, 45.2)
- added C5: 100nF, Capacitor_SMD:C_0402_1005Metric, F.Cu at (96.5, 63.7)
- added C6: 100nF, Capacitor_SMD:C_0402_1005Metric, F.Cu at (98.0, 63.2)
- added C7: 100nF, Capacitor_SMD:C_0402_1005Metric, F.Cu at (86.2, 63.5)
- added C8: 100nF, Capacitor_SMD:C_0402_1005Metric, F.Cu at (100.5, 55.2)
- added C9: 22uF, Capacitor_SMD:C_0805_2012Metric, F.Cu at (53.5, 50.8)
- added D1: LED, LED_SMD:LED_0603_1608Metric, F.Cu at (120.0, 36.5)
- added J1: ISP, Connector_IDC:IDC-Header_2x03_P2.54mm_Vertical, F.Cu at (118.0, 46.7)
- added J3: UART, Connector_PinHeader_2.54mm:PinHeader_1x06_P2.54mm_Vertical, F.Cu at (128.2, 55.5)
- added J4: OLED SSD1306, Connector_PinHeader_2.54mm:PinHeader_1x04_P2.54mm_Vertical, F.Cu at (135.7, 37.7)
- added J5: Drive_Power, TerminalBlock_RND:TerminalBlock_RND_205-00003_1x04_P5.00mm_Horizontal, F.Cu at (58.2, 30.0)
- added J6: 12V DC-In, ATAPIMega:BarrelJack_DC-005-2.0_C16214, F.Cu at (49.2, 63.0)
- added J7: External buttons, Connector_PinHeader_2.54mm:PinHeader_1x08_P2.54mm_Vertical, F.Cu at (74.7, 94.2)
- added J8: 3.5mm, Connector_Audio:Jack_3.5mm_CUI_SJ1-3535NG_Horizontal, F.Cu at (47.0, 119.7)
- added J9: Audio in, Connector_PinHeader_2.54mm:PinHeader_1x04_P2.54mm_Vertical, F.Cu at (126.0, 27.2)
- added L1: 4.7uH, Inductor_SMD:L_Bourns_SRP7028A_7.3x6.6mm, F.Cu at (64.5, 49.7)
- added R1: 10k, Resistor_SMD:R_0402_1005Metric, F.Cu at (99.7, 43.7)
- added R10: 30k, Resistor_SMD:R_0603_1608Metric, F.Cu at (58.9, 53.7)
- added R16: 10k, Resistor_SMD:R_0402_1005Metric, F.Cu at (105.0, 37.0)
- added R18: 10k, Resistor_SMD:R_0402_1005Metric, F.Cu at (92.2, 37.0)
- added R2: 75R, Resistor_SMD:R_0402_1005Metric, F.Cu at (101.2, 74.0)
- added R3: 4.7k, Resistor_SMD:R_0402_1005Metric, F.Cu at (116.2, 36.5)
- added R4: 4.7k, Resistor_SMD:R_0402_1005Metric, F.Cu at (128.0, 34.5)
- added R5: 4.7k, Resistor_SMD:R_0402_1005Metric, F.Cu at (130.7, 34.5)
- added R6: 10k, Resistor_SMD:R_0402_1005Metric, F.Cu at (69.5, 36.7)
- added R7: 10k, Resistor_SMD:R_0402_1005Metric, F.Cu at (99.7, 37.0)
- added R8: 75R, Resistor_SMD:R_0402_1005Metric, F.Cu at (101.7, 43.7)
- added R9: 220k, Resistor_SMD:R_0603_1608Metric, F.Cu at (55.9, 53.7)
- added RN1: 33R, Resistor_SMD:R_Array_Convex_4x0402, F.Cu at (92.0, 43.0)
- added RN2: 33R, Resistor_SMD:R_Array_Convex_4x0402, F.Cu at (101.0, 58.0)
- added RN3: 33R, Resistor_SMD:R_Array_Convex_4x0402, F.Cu at (89.5, 43.0)
- added RN4: 33R, Resistor_SMD:R_Array_Convex_4x0402, F.Cu at (81.0, 50.0)
- added RN5: 33R, Resistor_SMD:R_Array_Convex_4x0402, F.Cu at (91.0, 64.5)
- added RN6: 33R, Resistor_SMD:R_Array_Convex_4x0402, F.Cu at (88.5, 64.5)
- added RV1: 10k Contrast, Potentiometer_THT:Potentiometer_Bourns_3296W_Vertical, F.Cu at (65.7, 72.0)
- added SW1: Rew, Button_Switch_SMD:SW_Push_1P1T_NO_6x6mm_H9.5mm, F.Cu at (68.2, 118.0)
- added SW2: Prev, Button_Switch_SMD:SW_Push_1P1T_NO_6x6mm_H9.5mm, F.Cu at (55.7, 118.0)
- added SW3: Play/Pause, Button_Switch_SMD:SW_Push_1P1T_NO_6x6mm_H9.5mm, F.Cu at (80.7, 118.0)
- added SW4: Fwd, Button_Switch_SMD:SW_Push_1P1T_NO_6x6mm_H9.5mm, F.Cu at (93.2, 118.0)
- added SW5: Next, Button_Switch_SMD:SW_Push_1P1T_NO_6x6mm_H9.5mm, F.Cu at (105.7, 118.0)
- added SW6: Stop/Eject, Button_Switch_SMD:SW_Push_1P1T_NO_6x6mm_H9.5mm, F.Cu at (118.2, 118.0)
- added SW7: Shuffle/Repeat, Button_Switch_SMD:SW_Push_1P1T_NO_6x6mm_H9.5mm, F.Cu at (130.7, 118.0)
- added U1: ATmega2560-16AU, Package_QFP:TQFP-100_14x14mm_P0.5mm, F.Cu at (91.1, 54.0)
- added U2: HD44780, Display:WC1602A, F.Cu at (65.7, 78.0)
- added U3: SY8113B, Package_TO_SOT_SMD:TSOT-23-6, F.Cu at (58.5, 50.7)
- added Y1: 16 MHz, Crystal:Crystal_SMD_3225-4Pin_3.2x2.5mm, F.Cu at (96.5, 42.2)
- moved H2 163.5 mm to (39.2, 26.5)
- moved J2 141.8 mm to (67.5, 31.7), turned to 90 degrees
- moved H1 83.3 mm to (137.2, 124.5)
Connections:
- J2 pad 10: /D11 -> Net-(J2-Pad10)
- J2 pad 11: /D3 -> Net-(J2-Pad11)
- J2 pad 12: /D12 -> Net-(J2-Pad12)
- J2 pad 13: /D2 -> Net-(J2-Pad13)
- J2 pad 14: /D13 -> Net-(J2-Pad14)
- J2 pad 15: /D1 -> Net-(J2-Pad15)
- J2 pad 16: /D14 -> Net-(J2-Pad16)
- J2 pad 17: /D0 -> Net-(J2-Pad17)
- J2 pad 18: /D15 -> Net-(J2-Pad18)
- J2 pad 21: /DMA_RQ -> /ATA_DMA_RQ
- J2 pad 23: /IOW -> Net-(J2-Pad23)
- J2 pad 25: /IOR -> Net-(J2-Pad25)
- J2 pad 27: /IO_CH_RD -> /ATA_IO_CH_RD
- J2 pad 3: /D7 -> /ATA_D7
- J2 pad 31: /IRQ -> /ATA_IRQ
- J2 pad 33: /DA1 -> Net-(J2-Pad33)
- J2 pad 35: /DA0 -> Net-(J2-Pad35)
- J2 pad 37: /CS0 -> Net-(J2-Pad37)
- J2 pad 4: /D8 -> Net-(J2-Pad4)
- J2 pad 5: /D6 -> Net-(J2-Pad5)
- J2 pad 6: /D9 -> Net-(J2-Pad6)
- J2 pad 7: /D5 -> Net-(J2-Pad7)
- J2 pad 8: /D10 -> Net-(J2-Pad8)
- J2 pad 9: /D4 -> Net-(J2-Pad9)
Routing:
- net Net-(J8-PadS): track 0.00 -> 170.0 mm
- net Net-(J8-PadT): track 0.00 -> 164.7 mm, vias 0 -> 1
- net Net-(J8-PadR): track 0.00 -> 161.6 mm
- net /BTN_SHUFFLE: track 0.00 -> 96.9 mm, vias 0 -> 2
- net /BTN_STOP: track 0.00 -> 90.9 mm, vias 0 -> 2
- net /BTN_NEXT: track 0.00 -> 79.0 mm, vias 0 -> 2
- net /BTN_FWD: track 0.00 -> 78.6 mm, vias 0 -> 2
- net /BTN_PREV: track 0.00 -> 76.0 mm, vias 0 -> 2
- net /BTN_PLAY: track 0.00 -> 72.1 mm, vias 0 -> 2
- net GND: track 0.00 -> 71.4 mm, vias 0 -> 184
- net /BTN_REW: track 0.00 -> 69.9 mm, vias 0 -> 2
- net +5V: track 0.00 -> 60.2 mm, vias 0 -> 18
- net Net-(J2-Pad4): track 0.00 -> 56.0 mm, vias 0 -> 1
- net Net-(J2-Pad6): track 0.00 -> 53.8 mm, vias 0 -> 1
- net /OLED_SCL: track 0.00 -> 53.3 mm, vias 0 -> 3
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- added copper zone on In2.Cu, net +12V
- added copper zone on In2.Cu, net +5V
- added copper zone on B.Cu, net GND
- added copper zone on F.Cu, net GND
Other:
- board outline added: 100 x 100 mm
- copper layers 2 -> 4
- net class Default: via_dia 0.6 -> 0.4; via_drill 0.3 -> 0.2
- rule via_min_drill: 0.3 -> 0.2
- rule via_min_size: 0.6 -> 0.4
- board text added: "*meow*"
- board text added: "1"
- board text added: "12V"
- board text added: "12V DC"
- board text added: "5V"
- board text added: "ATAPI Audio-CD Player"
- board text added: "ATAPI Interface"
- board text added: "Audio in"
- board text added: "CTS"
- board text added: "DTR"
- board text added: "Drive power"
- board text added: "GND"
- board text added: "I2C"
- board text added: "ISP"
- board text added: "LCD Contrast"
- board text added: "RX"
- board text added: "SDA SCL 5V GND"
- board text added: "TX"
- board text added: "UART"

Commit message: PCB
Parts:
- added C2: 100nF, Capacitor_SMD:C_0402_1005Metric, F.Cu at (81.7, 53.5)
- added H3: Catboy, ATAPIMega:catboy, B.Cu at (92.0, 54.0)
- moved J8 2.01 mm to (46.8, 121.7)
Connections:
- J6 pad 3: Net-(J6-Pad3) -> GND
Routing:
- net GND: track 71.4 -> 79.0 mm, vias 184 -> 205
- net +12V: track 47.7 -> 51.2 mm
- net /RESET: track 38.8 -> 36.6 mm, vias 2 -> 0
- net Net-(J8-PadT): track 164.7 -> 166.7 mm
- net +5V: track 60.2 -> 61.9 mm
- net Net-(J8-PadS): track 170.0 -> 171.4 mm
- net /LCD_D1: track 24.0 -> 22.6 mm
- net Net-(J8-PadR): track 161.6 -> 162.7 mm
- net /LCD_D2: track 21.9 -> 21.0 mm
- net /LCD_D0: track 26.3 -> 27.2 mm
- added copper zone on In1.Cu, net GND
Other:
- net class Default: via_dia 0.4 -> 0.45
- rule via_min_size: 0.4 -> 0.45
- board text added: "Rev.A 2021 Tobias Mädel / Tobias Schramm"
- board text added: "tbspace.de"

Commit message: RevA
Routing:
- net +5V: track 61.9 -> 63.4 mm
- net /IRQ: track 20.0 -> 21.4 mm
- net Net-(J8-PadR): track 162.7 -> 164.0 mm
- net /CS0: track 22.4 -> 23.6 mm
- net Net-(J2-Pad12): track 49.2 -> 50.2 mm
- net /DA2: track 41.9 -> 42.9 mm
- net Net-(J2-Pad4): track 56.0 -> 55.4 mm
- net /LCD_D4: vias 1 -> 0
